File: V0/V0.4/EDA/daughter_board/KiCAD_v3/Magdron mount.kicad_pcb (KiCad board)
At the start: 2 copper layers, 40 x 40 mm, 18 parts, among them U4 top_rail_v2

Commit message: major cleanup
Other:
- board text added: "DB V0.4"
- board text removed: "DB V1.8"
