File: V0/V0.4/EDA/main_board/main_board.kicad_pcb (KiCad board)
At the start: 2 copper layers, 40.6 x 78.5 mm, 28 parts, among them U1 top_rail_v2, U2 DS3231M, U3 INA219AxD, U5 KA78M05_TO252

Commit message: major cleanup
Parts:
- ARDUINO NANO: renamed from A1
- MICRO SD: renamed from Micro_SD1
- renumbered U5 to 5V, BT1 to CR-1025, U2 to DS3231, Power_IN1 to POWER, Ultrasonic_sensor1 to STAGE
Other:
- board text added: "MB V0.4"
- board text removed: "DEBUG"
- board text removed: "DEPLOY"
- board text removed: "MB V1.8"
