File: system_design/Georgetown/V0.5.2/EDA/main_board/main_board.kicad_sch (KiCad schematic)
At the start: 34 parts, among them J1 B3B-XH-A_LF__SN_, J2 Conn_01x02_Pin, P1 SD card socket, Q1 MMBT2222A, SW1 SW_Wuerth_450301014042, U1 HX-2S-JH10, U2 DS3231M, U4 BME280_module, U5 KA78M05_TO252

Commit message: BOM updated
Parts:
- U3: value ~ -> psw03c
Changed lines of the file:
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@@
 			)
 		)
-		(property "Value" "~"
+		(property "Value" "psw03c"
 			(at 170.815 48.26 0)
 			(effects
